Commit message: Removed cmd_vel clamp and switched run time to sim time.

File: adeept_awr/adeept_awr_description/urdf/adeept_awr.urdf (robot description, URDF)
Before this commit: robot adeept_awr, 7 links, 6 joints
Links:
- link chassis: mass 0.500 -> None

Commit message: Update map terrain * Added uneven terrain. * Spawn robot from lower height. * Zoom out GUI camera to see full playing field. * Rebalance the robot to stop it from tipping over.

File: adeept_awr/adeept_awr_description/urdf/adeept_awr.urdf (robot description, URDF)
Before this commit: robot adeept_awr, 7 links, 6 joints
Links:
- link battery: mass 0.230 -> 0.005
